File: hardware/sp0256_dcf77.brd (EAGLE design)
At the start: 151.4 x 117.5 mm, 83 parts, among them IC1 74245N, IC2 MAX232, IC3 LM386N-1, IC5 ATF16V8BP3, IC7 7805T

Commit message: PCB updated
Connections:
- removed net DCF77_PULSE_IN: IC11.26, JP4.2
- new net !DCF77_PULSE: IC11.26, IC5.15
- new net DCF77_PULSE: IC5.8, JP4.2
Routing:
- net DCF77_PULSE: track 0.00 -> 86.2 mm, vias 0 -> 2
- net !DCF77_PULSE: track 0.00 -> 51.4 mm, vias 0 -> 2
- net DCF77_PULSE_IN: track 33.3 -> 0.00 mm
- net CS_0: track 79.6 -> 80.5 mm
- net A9: track 108.1 -> 108.7 mm
- net A8: track 109.4 -> 109.9 mm
Changed lines of the file:
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@@
 <wire x1="115.8875" y1="17.145" x2="114.935" y2="17.145" width="0.4064" layer="16"/>
 <wire x1="114.935" y1="17.145" x2="112.395" y2="19.685" width="0.4064" layer="16"/>
-<wire x1="109.22" y1="33.02" x2="103.505" y2="33.02" width="0.4064" layer="16"/>
+<wire x1="109.855" y1="33.02" x2="103.505" y2="33.02" width="0.4064" layer="16"/>
 <wire x1="103.505" y1="33.02" x2="99.3775" y2="37.1475" width="0.4064" layer="16"/>
 <wire x1="99.3775" y1="37.1475" x2="96.8375" y2="37.1475" width="0.4064" layer="16"/>
@@
 <wire x1="112.395" y1="19.685" x2="112.395" y2="21.2725" width="0.4064" layer="16"/>
 <wire x1="112.395" y1="21.2725" x2="111.4425" y2="22.225" width="0.4064" layer="16"/>
-<wire x1="111.4425" y1="22.225" x2="111.4425" y2="23.495" width="0.4064" layer="16"/>
-<wire x1="111.4425" y1="23.495" x2="110.49" y2="24.4475" width="0.4064" layer="16"/>
-<wire x1="110.49" y1="24.4475" x2="110.49" y2="25.7175" width="0.4064" layer="16"/>
-<wire x1="109.22" y1="33.02" x2="109.855" y2="32.385" width="0.4064" layer="16"/>
-<wire x1="109.855" y1="32.385" x2="109.855" y2="26.3525" width="0.4064" layer="16"/>
-<wire x1="109.855" y1="26.3525" x2="110.49" y2="25.7175" width="0.4064" layer="16"/>
+<wire x1="111.4425" y1="22.225" x2="111.4425" y2="31.4325" width="0.4064" layer="16"/>
+<wire x1="111.4425" y1="31.4325" x2="109.855" y2="33.02" width="0.4064" layer="16"/>
 </signal>
 <signal name="IRQ">
@@
 <wire x1="109.22" y1="11.43" x2="109.22" y2="15.24" width="0.4064" layer="16"/>
 <wire x1="109.22" y1="15.24" x2="106.68" y2="17.78" width="0.4064" layer="16"/>
-<wire x1="106.68" y1="17.78" x2="102.235" y2="17.78" width="0.4064" layer="16"/>
-<wire x1="102.235" y1="17.78" x2="100.965" y2="19.05" width="0.4064" layer="16"/>
-<wire x1="100.965" y1="19.05" x2="97.79" y2="19.05" width="0.4064" layer="16"/>
+<wire x1="106.68" y1="17.78" x2="104.14" y2="17.78" width="0.4064" layer="16"/>
+<wire x1="104.14" y1="17.78" x2="102.87" y2="19.05" width="0.4064" layer="16"/>
+<wire x1="102.87" y1="19.05" x2="97.79" y2="19.05" width="0.4064" layer="16"/>
 </signal>
 <signal name="RW">
@@
 <wire x1="113.03" y1="12.7" x2="113.03" y2="16.51" width="0.4064" layer="16"/>
 <wire x1="113.03" y1="16.51" x2="110.49" y2="19.05" width="0.4064" layer="16"/>
-<wire x1="106.9975" y1="27.94" x2="102.235" y2="27.94" width="0.4064" layer="16"/>
+<wire x1="107.95" y1="27.94" x2="102.235" y2="27.94" width="0.4064" layer="16"/>
 <wire x1="102.235" y1="27.94" x2="100.965" y2="29.21" width="0.4064" layer="16"/>
 <wire x1="100.965" y1="29.21" x2="97.79" y2="29.21" width="0.4064" layer="16"/>
 <wire x1="110.49" y1="19.05" x2="110.49" y2="20.6375" width="0.4064" layer="16"/>
 <wire x1="110.49" y1="20.6375" x2="109.5375" y2="21.59" width="0.4064" layer="16"/>
-<wire x1="109.5375" y1="21.59" x2="109.5375" y2="22.86" width="0.4064" layer="16"/>
-<wire x1="109.5375" y1="22.86" x2="108.585" y2="23.8125" width="0.4064" layer="16"/>
-<wire x1="108.585" y1="23.8125" x2="108.585" y2="25.0825" width="0.4064" layer="16"/>
-<wire x1="107.6325" y1="26.035" x2="107.6325" y2="27.305" width="0.4064" layer="16"/>
-<wire x1="107.6325" y1="27.305" x2="106.9975" y2="27.94" width="0.4064" layer="16"/>
-<wire x1="108.585" y1="25.0825" x2="107.6325" y2="26.035" width="0.4064" layer="16"/>
+<wire x1="107.95" y1="27.94" x2="109.5375" y2="26.3525" width="0.4064" layer="16"/>
+<wire x1="109.5375" y1="21.59" x2="109.5375" y2="26.3525" width="0.4064" layer="16"/>
 </signal>
 <signal name="A9">
@@
 <wire x1="112.0775" y1="16.1925" x2="109.5375" y2="18.7325" width="0.4064" layer="16"/>
 <contactref element="IC5" pad="4"/>
-<wire x1="106.9975" y1="25.4" x2="102.235" y2="25.4" width="0.4064" layer="16"/>
+<wire x1="107.95" y1="25.4" x2="102.235" y2="25.4" width="0.4064" layer="16"/>
 <wire x1="102.235" y1="25.4" x2="100.965" y2="26.67" width="0.4064" layer="16"/>
 <wire x1="100.965" y1="26.67" x2="97.79" y2="26.67" width="0.4064" layer="16"/>
 <wire x1="109.5375" y1="18.7325" x2="109.5375" y2="20.32" width="0.4064" layer="16"/>
 <wire x1="109.5375" y1="20.32" x2="108.585" y2="21.2725" width="0.4064" layer="16"/>
-<wire x1="108.585" y1="21.2725" x2="108.585" y2="22.5425" width="0.4064" layer="16"/>
-<wire x1="108.585" y1="22.5425" x2="107.6325" y2="23.495" width="0.4064" layer="16"/>
-<wire x1="107.6325" y1="23.495" x2="107.6325" y2="24.765" width="0.4064" layer="16"/>
-<wire x1="107.6325" y1="24.765" x2="106.9975" y2="25.4" width="0.4064" layer="16"/>
+<wire x1="107.95" y1="25.4" x2="108.585" y2="24.765" width="0.4064" layer="16"/>
+<wire x1="108.585" y1="24.765" x2="108.585" y2="21.2725" width="0.4064" layer="16"/>
 </signal>
 <signal name="A10">
@@
 <wire x1="97.79" y1="31.75" x2="102.235" y2="31.75" width="0.4064" layer="16"/>
 <wire x1="102.235" y1="31.75" x2="103.505" y2="30.48" width="0.4064" layer="16"/>
-<wire x1="103.505" y1="30.48" x2="106.9975" y2="30.48" width="0.4064" layer="16"/>
+<wire x1="103.505" y1="30.48" x2="108.585" y2="30.48" width="0.4064" layer="16"/>
 <wire x1="111.4425" y1="19.3675" x2="114.935" y2="15.875" width="0.4064" layer="16"/>
 <wire x1="111.4425" y1="19.3675" x2="111.4425" y2="20.955" width="0.4064" layer="16"/>
 <wire x1="111.4425" y1="20.955" x2="110.49" y2="21.9075" width="0.4064" layer="16"/>
-<wire x1="110.49" y1="21.9075" x2="110.49" y2="23.1775" width="0.4064" layer="16"/>
-<wire x1="110.49" y1="23.1775" x2="109.5375" y2="24.13" width="0.4064" layer="16"/>
-<wire x1="109.5375" y1="24.13" x2="109.5375" y2="25.4" width="0.4064" layer="16"/>
-<wire x1="109.5375" y1="25.4" x2="108.585" y2="26.3525" width="0.4064" layer="16"/>
-<wire x1="108.585" y1="26.3525" x2="108.585" y2="28.8925" width="0.4064" layer="16"/>
-<wire x1="108.585" y1="28.8925" x2="106.9975" y2="30.48" width="0.4064" layer="16"/>
+<wire x1="110.49" y1="21.9075" x2="110.49" y2="28.575" width="0.4064" layer="16"/>
+<wire x1="110.49" y1="28.575" x2="108.585" y2="30.48" width="0.4064" layer="16"/>
 </signal>
 <signal name="CS_1">
@@
 <wire x1="126.6825" y1="45.085" x2="118.11" y2="45.085" width="0.4064" layer="16"/>
 <wire x1="118.11" y1="45.085" x2="116.84" y2="46.355" width="0.4064" layer="16"/>
-<wire x1="116.84" y1="46.355" x2="108.585" y2="46.355" width="0.4064" layer="16"/>
-<via x="108.585" y="46.355" extent="1-16" drill="0.6" diameter="1.4224" shape="octagon"/>
+<wire x1="116.84" y1="46.355" x2="109.22" y2="46.355" width="0.4064" layer="16"/>
+<via x="109.22" y="46.355" extent="1-16" drill="0.6" diameter="1.4224" shape="octagon"/>
 <contactref element="IC5" pad="19"/>
-<wire x1="105.41" y1="31.75" x2="108.585" y2="31.75" width="0.4064" layer="16"/>
-<via x="108.585" y="31.75" extent="1-16" drill="0.6" diameter="1.4224" shape="octagon"/>
-<wire x1="108.585" y1="31.75" x2="108.585" y2="46.355" width="0.4064" layer="1"/>
+<wire x1="105.41" y1="31.75" x2="109.22" y2="31.75" width="0.4064" layer="16"/>
+<via x="109.22" y="31.75" extent="1-16" drill="0.6" diameter="1.4224" shape="octagon"/>
+<wire x1="109.22" y1="31.75" x2="109.22" y2="46.355" width="0.4064" layer="1"/>
 </signal>
 <signal name="TIMER_CS">
 <contactref element="IC11" pad="15"/>
-<via x="102.87" y="40.005" extent="1-16" drill="0.6" diameter="1.4224" shape="octagon"/>
-<wire x1="102.87" y1="40.005" x2="105.41" y2="40.005" width="0.6096" layer="16"/>
+<via x="107.95" y="40.005" extent="1-16" drill="0.6" diameter="1.4224" shape="octagon"/>
 <contactref element="IC5" pad="18"/>
-<wire x1="105.41" y1="29.21" x2="102.87" y2="29.21" width="0.4064" layer="16"/>
-<via x="102.87" y="29.21" extent="1-16" drill="0.6" diameter="1.4224" shape="octagon"/>
-<wire x1="102.87" y1="29.21" x2="102.87" y2="40.005" width="0.4064" layer="1"/>
+<wire x1="105.41" y1="29.21" x2="107.95" y2="29.21" width="0.4064" layer="16"/>
+<via x="107.95" y="29.21" extent="1-16" drill="0.6" diameter="1.4224" shape="octagon"/>
+<wire x1="107.95" y1="29.21" x2="107.95" y2="40.005" width="0.4064" layer="1"/>
+<wire x1="107.95" y1="40.005" x2="105.41" y2="40.005" width="0.6096" layer="16"/>
 </signal>
 <signal name="GATE2">
@@
 <wire x1="90.17" y1="70.485" x2="92.495" y2="70.485" width="0.6096" layer="16"/>
 </signal>
-<signal name="DCF77_PULSE_IN">
-<contactref element="IC11" pad="26"/>
-<wire x1="105.41" y1="67.945" x2="104.14" y2="67.945" width="0.4064" layer="16"/>
-<wire x1="104.14" y1="67.945" x2="103.1875" y2="68.8975" width="0.4064" layer="16"/>
-<wire x1="103.1875" y1="68.8975" x2="103.1875" y2="75.2475" width="0.4064" layer="16"/>
-<wire x1="103.1875" y1="75.2475" x2="101.6" y2="76.835" width="0.4064" layer="16"/>
+<signal name="DCF77_PULSE">
 <wire x1="101.6" y1="76.835" x2="88.5825" y2="76.835" width="0.4064" layer="16"/>
 <contactref element="JP4" pad="2"/>
 <wire x1="86.6775" y1="85.09" x2="86.6775" y2="78.74" width="0.4064" layer="16"/>
 <wire x1="86.6775" y1="78.74" x2="88.5825" y2="76.835" width="0.4064" layer="16"/>
+<contactref element="IC5" pad="8"/>
+<via x="101.6" y="76.835" extent="1-16" drill="0.6" diameter="1.4224"/>
+<wire x1="101.6" y1="76.835" x2="101.6" y2="16.51" width="0.4064" layer="1"/>
+<via x="101.6" y="16.51" extent="1-16" drill="0.6" diameter="1.4224" shape="octagon"/>
+<wire x1="101.6" y1="16.51" x2="97.79" y2="16.51" width="0.4064" layer="16"/>
 </signal>
 <signal name="N$27">
@@
 <wire x1="116.5225" y1="84.455" x2="118.8475" y2="84.455" width="0.6096" layer="16"/>
 </signal>
+<signal name="!DCF77_PULSE">
+<contactref element="IC5" pad="15"/>
+<contactref element="IC11" pad="26"/>
+<wire x1="105.41" y1="21.59" x2="102.87" y2="21.59" width="0.4064" layer="16"/>
+<via x="102.87" y="21.59" extent="1-16" drill="0.6" diameter="1.4224" shape="octagon"/>
+<wire x1="102.87" y1="21.59" x2="102.87" y2="67.945" width="0.4064" layer="1"/>
+<via x="102.87" y="67.945" extent="1-16" drill="0.6" diameter="1.4224" shape="octagon"/>
+<wire x1="102.87" y1="67.945" x2="105.41" y2="67.945" width="0.4064" layer="16"/>
+</signal>
 </signals>
